File: dm13a-breakout-board.kicad_pcb (KiCad board)
At the start: 2 copper layers, 0 parts

Commit message: Try the whole thing
Parts:
- added C1: 0.1uF, Capacitor_SMD:C_0603_1608Metric, F.Cu at (81.0, 58.2)
- added H1: MountingHole, MountingHole:MountingHole_3.2mm_M3, F.Cu at (55.0, 55.0)
- added H2: MountingHole, MountingHole:MountingHole_3.2mm_M3, F.Cu at (95.0, 55.0)
- added H3: MountingHole, MountingHole:MountingHole_3.2mm_M3, F.Cu at (55.0, 95.0)
- added H4: MountingHole, MountingHole:MountingHole_3.2mm_M3, F.Cu at (95.0, 95.0)
- added J1: Conn_01x02, Connector_PinHeader_2.54mm:PinHeader_1x02_P2.54mm_Vertical, F.Cu at (84.2, 54.5)
- added J2: Conn_01x05, Connector_PinHeader_2.54mm:PinHeader_1x05_P2.54mm_Vertical, F.Cu at (68.9, 54.5)
- added J3: Conn_01x08, Connector_PinHeader_2.54mm:PinHeader_1x08_P2.54mm_Vertical, F.Cu at (63.0, 70.9)
- added J4: Conn_01x08, Connector_PinHeader_2.54mm:PinHeader_1x08_P2.54mm_Vertical, F.Cu at (87.0, 70.9)
- added R1: 5k, Resistor_THT:R_Axial_DIN0411_L9.9mm_D3.6mm_P12.70mm_Horizontal, F.Cu at (96.3, 63.5)
- added U1: DM13A, Package_DIP:DIP-24_W7.62mm, F.Cu at (70.9, 60.8)
Routing:
- net /LATCH: track 0.00 -> 15.2 mm
- net /BRIGHTNESS: track 0.00 -> 14.8 mm
- net /CLOCK: track 0.00 -> 12.3 mm
- net /DATA: track 0.00 -> 9.71 mm
- net +5V: track 0.00 -> 9.10 mm
- net Net-(J4-Pin_2): track 0.00 -> 8.53 mm
- net Net-(J4-Pin_8): track 0.00 -> 8.53 mm
- net Net-(J4-Pin_7): track 0.00 -> 8.53 mm
- net Net-(J4-Pin_6): track 0.00 -> 8.53 mm
- net Net-(J4-Pin_5): track 0.00 -> 8.53 mm
- net Net-(J4-Pin_4): track 0.00 -> 8.53 mm
- net Net-(J4-Pin_3): track 0.00 -> 8.53 mm
- net Net-(J4-Pin_1): track 0.00 -> 8.53 mm
- net Net-(J3-Pin_3): track 0.00 -> 7.93 mm
- net Net-(J3-Pin_1): track 0.00 -> 7.93 mm
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- added copper zone on B.Cu, net GND
- added copper zone on F.Cu, net GND
Other:
- board outline added: 50 x 50 mm
- board text added: "${VERSION} ${DATE}"
